File: display/display.kicad_pcb (KiCad board)
At the start: 2 copper layers, 26 parts, among them J1 IO out, J2 IO in, Q1 2N3906, Q2 2N3906, Q3 2N3906, Q4 2N3906, U1 74HC14, U10 74HCT574, U11 ATA8401ARBJ, U2 74LS139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

Commit message: display pcb first version ready
Parts:
- added H1: MountingHole, MountingHole:MountingHole_2.2mm_M2, F.Cu at (158.6, 123.8)
- added H2: MountingHole, MountingHole:MountingHole_2.2mm_M2, F.Cu at (80.3, 55.4)
Routing:
- net /S8: track 118.5 -> 166.1 mm, vias 1 -> 2
- net /S5: track 116.3 -> 156.5 mm
- net /S6: track 115.0 -> 154.1 mm, vias 1 -> 3
- net /S3: track 114.8 -> 153.8 mm, vias 1 -> 3
- net /S7: track 115.9 -> 154.8 mm, vias 1 -> 3
- net /S4: track 118.6 -> 156.8 mm, vias 1 -> 3
- net Net-(U4-Pad13): track 48.3 -> 58.4 mm
- net /~OE3: track 65.5 -> 69.6 mm
- net VCC: track 304.4 -> 306.6 mm
- net /DDg1: track 46.7 -> 48.5 mm, vias 1 -> 2
- net /~OE2: track 107.6 -> 108.6 mm
- net /I4: track 226.2 -> 225.5 mm
- net /I5: track 204.7 -> 204.0 mm
- net /I6: track 202.6 -> 201.9 mm
- net /I3: track 228.2 -> 227.6 mm
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- added copper zone on B.Cu, net GND
- added copper zone on F.Cu, net GND
Other:
- board outline added: 112.4 x 78.7 mm
- board text added: "+5V"
- board text added: "0"
- board text added: "7"
- board text added: "Address I/O"
- board text added: "Data I/0"
- board text added: "GND"
- board text added: "~INT"
- board text added: "~INTCK"
- board text added: "~IOREAD"
- board text added: "~IOWRT"
- board text added: "~WAIT"
