File: tangentbord/tangentbord.sch (KiCad schematic (older format))
At the start: 59 parts

Commit message: Tangentbord pcb v1
Parts:
- removed R?: 4k7, symbol Device:R
- removed SW?: SW_Push, symbol Switch:SW_Push
- removed U?: 74HC14, symbol 74xx:74HC14
- removed U?: 74LS273, symbol 74xx:74LS273
- removed U?: 74LS540, symbol 74xx:74LS540
- added C1: 10u, Capacitor_THT:CP_Radial_D5.0mm_P2.00mm, symbol Device:CP
- added C2: 47n, Capacitor_THT:C_Disc_D3.0mm_W2.0mm_P2.50mm, symbol Device:C
- added D1: LED, LED_THT:LED_D3.0mm, symbol Device:LED
- added H1, H2, H3: MountingHole, MountingHole:MountingHole_2.2mm_M2, symbol Mechanical:MountingHole
- added R12, R13: 4k7, Resistor_THT:R_Axial_DIN0207_L6.3mm_D2.5mm_P7.62mm_Horizontal, symbol Device:R
- added SW31, SW32, SW33, SW34: SW_Push_45deg, Button_Switch_THT:SW_PUSH_6mm, symbol Switch:SW_Push_45deg
- added unit 5 of U1
- added unit 6 of U1
- added U3: 4071, Package_DIP:DIP-14_W7.62mm, symbol 4xxx:4071
- added U4: 74HC4078, Package_DIP:DIP-14_W7.62mm, symbol 74xx:74HC4078
- added U6, U7: 74LS574, Package_DIP:DIP-20_W7.62mm, symbol 74xx:74LS574
- C3, C4: renamed from C?; footprint (none) -> Capacitor_THT:C_Disc_D3.0mm_W2.0mm_P2.50mm
- J1: renamed from J?; footprint (none) -> Connector_PinHeader_2.54mm:PinHeader_1x24_P2.54mm_Vertical
- R1, R10, R11, R2, R3, R4, R5, R6, R7, R8, R9: renamed from R?; footprint (none) -> Resistor_THT:R_Axial_DIN0207_L6.3mm_D2.5mm_P7.62mm_Horizontal
- SW1, SW10, SW11, SW12, SW13, SW14, SW15, SW16, SW17, SW18, SW19, SW2, SW20, SW21, SW22, SW23, SW24, SW25, SW26, SW27, SW28, SW29, SW3, SW30, SW4, SW5, SW6, SW7, SW8, SW9: renamed from SW?; footprint (none) -> Button_Switch_THT:SW_PUSH_6mm
- U1, U5: renamed from U?; footprint (none) -> Package_DIP:DIP-14_W7.62mm
- U2, U8: renamed from U?; footprint (none) -> Package_DIP:DIP-16_W7.62mm
Connections:
- net SK3 is gone; now on net SK2: R2.2, SW2.2
- net A0: now also U1.13, U3.6; no longer U2.2 (A0), U5.4 (Q1)
- net A1: now also U4.11 (G); no longer U2.3 (A1), U5.3 (Q0)
- net A2: now also U1.11
- net A3: now also U4.2 (A)
- net A4: now also U4.3 (B)
- net A5: now also U4.4 (C)
- net A6: now also U4.5 (D)
- net A7: now also U4.9 (E)
- net GND: now also U8.5 (EI), C1.2, C2.2, R13.2, U3.7 (VSS), U4.7 (GND), U6.10 (GND), U7.10 (GND)
- net I0: now also U6.12 (Q7), U7.12 (Q7)
- net I1: now also U6.13 (Q6), U7.13 (Q6)
- net I2: now also U6.14 (Q5), U7.14 (Q5)
- net I3: now also U6.15 (Q4), U7.15 (Q4)
- net I4: now also U6.16 (Q3), U7.16 (Q3)
- net I5: now also U6.17 (Q2), U7.17 (Q2)
- net I6: now also U6.18 (Q1), U7.18 (Q1)
- net I7: now also U6.19 (Q0), U7.19 (Q0)
- net R1: now also SW31.2
- net R2: now also SW32.2
- net R3: now also SW33.2
- net R4: now also SW34.2
- net S0: now also U6.4 (D2), U7.4 (D2)
- net S1: now also U6.5 (D3), U7.5 (D3)
- net S2: now also U6.6 (D4), U7.6 (D4)
- net SK1: now also R1.2, SW1.2, U6.2 (D0), U7.2 (D0)
- net SK2: now also U6.3 (D1), U7.3 (D1); no longer R1.2, SW1.2
- net VCC: now also C1.1, C2.1, D1.2 (A), R12.1, U3.14 (VDD), U4.14 (VCC), U6.20 (VCC), U7.20 (VCC); no longer U8.4 (I7)
- net ~IOREAD: now also U4.12 (H)
- net at U8.14 (GS): now also U6.9 (D7), U7.9 (D7)
- net CPKP: now reaches U8.15 (EO)
- net CPKP: now also U6.11 (Cp)
- net CPKR: now reaches U1.6
- net CPKR: now also U7.11 (Cp)
- net at U1.9: now also R11.2, U1.2, U1.3
- removed net ~INEN: R11.2, U1.2, U1.3, U8.5 (EI)
- new net: U1.10, U4.10 (F)
- new net: U1.12, U3.2
- new net: D1.1 (K), R13.1
- new net AY: U3.1, U3.5, U4.1 (Y)
- new net L8: R12.2, SW31.1, SW32.1, SW33.1, SW34.1, U8.4 (I7)
- new net RN0: U2.2 (A0), U5.4 (Q1), U6.7 (D5), U7.7 (D5)
- new net RN1: U2.3 (A1), U5.3 (Q0), U6.8 (D6), U7.8 (D6)
- new net ~OE4: U3.4, U7.1 (OE)
- new net ~OE5: U3.3, U6.1 (OE)
- no-connect marks 2 -> 6
Other:
- note added: "Functions"
- note added: "Hex"
- note added: "Special Keys"
- moved on the sheet: U1B, U1G, U2A, U5A, U8
